File: hardware/kicad/J48_RevI.kicad_sch (KiCad schematic)
At the start: 86 parts, among them J1 ZIF-28, 0.3/0.6in, J2 USB-C 2.0 receptacle, J3 UPDI, J4 VSYS select 2x3, J5 Expansion 2x8, Q1 AO3400, Q2 BD139, Q3 BC547, Q4 AO3400, Q5 AO3400, Q6 AO3401, Q7 AO3401, SW1 latching push, U1 AVR16DU28-I/SP, U2 74HC595, U3 MCP4821-E/P, U4 MIC2288YD5, U6 LM358, U7 23LC1024-I/P, U8 LDL1117S33R, U9 74HC595

Commit message: Fix U1 pin numbers: use the SPDIP/SSOP-28 pinout
The reference schematic's AVR16DU28 symbol carried the VQFN-28 column of the
I/O multiplexing table instead of the SPDIP/SSOP-28 pinout, so every U1 pin
number was wrong. Pin numbers now follow DS40002576 section 2.4 (identical in
DS40002548 section 2.1 for the AVR64DU28), checked by script against the
datasheet text for all 28 pins. Pin positions are unchanged, so the drawing
and labels are unaffected.

Adds hardware/kicad/GALProg.kicad_sym with corrected AVR16DU28 and AVR64DU28
symbols for updating existing schematics in place.

Co-Authored-By: Claude Opus 5.5 <noreply@anthropic.com>
Claude-Session: https://claude.ai/code/session_01JnSUixWDwegCziKEySiVmX
Connections:
- net DAC_CS: now also U1.24 (PA2); no longer U1.28 (PA2)
- net GND: now also U1.15 (GND), U1.21 (GND); no longer U1.19 (GND), U1.25 (GND)
- net MCU_PA3: now also U1.25 (PA3); no longer U1.1 (PA3)
- net MCU_PC3: now also U1.5 (PC3); no longer U1.9 (PC3)
- net MCU_PD0: now also U1.6 (PD0); no longer U1.10 (PD0)
- net MCU_PD2: now also U1.8 (PD2); no longer U1.12 (PD2)
- net MCU_PD3: now also U1.9 (PD3); no longer U1.13 (PD3)
- net MCU_PD4: now also U1.10 (PD4); no longer U1.14 (PD4)
- net MCU_PD5: now also U1.11 (PD5); no longer U1.15 (PD5)
- net MCU_PD6: now also U1.12 (PD6); no longer U1.16 (PD6)
- net MCU_PD7: now also U1.13 (PD7); no longer U1.17 (PD7)
- net MCU_PF0: now also U1.16 (PF0); no longer U1.20 (PF0)
- net MCU_PF1: now also U1.17 (PF1); no longer U1.21 (PF1)
- net RESET: now also U1.18 (PF6/~{RESET}); no longer U1.22 (PF6/~{RESET})
- net SPI_MISO: now also U1.27 (PA5/MISO); no longer U1.3 (PA5/MISO)
- net SPI_MOSI: now also U1.26 (PA4/MOSI); no longer U1.2 (PA4/MOSI)
- net SPI_SCK: now also U1.28 (PA6/SCK); no longer U1.4 (PA6/SCK)
- net SRAM_CS: now also U1.22 (PA0); no longer U1.26 (PA0)
- net SR_OE: now also U1.23 (PA1); no longer U1.27 (PA1)
- net SR_RCLK: now also U1.1 (PA7); no longer U1.5 (PA7)
- net UPDI: now also U1.19 (PF7/UPDI); no longer U1.23 (PF7/UPDI)
- net USB_DM: now also U1.3 (DM); no longer U1.7 (DM)
- net USB_DP: now also U1.4 (DP); no longer U1.8 (DP)
- net VPP_SENSE: now also U1.7 (PD1/AIN1); no longer U1.11 (PD1/AIN1)
- net VSYS: now also U1.14 (VDD), U1.20 (VDD); no longer U1.18 (VDD), U1.24 (VDD)
- net VUSB: now also U1.2 (VUSB); no longer U1.6 (VUSB)
Changed lines of the file:
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@@
   (no_connect (at 30.48 254))
   (no_connect (at 207.01 356.87))
-  (symbol (lib_id "GALProg:AVR16DU28") (at 69.85 74.93 0) (unit 1) (exclude_from_sim no) (in_bom yes) (on_board yes) (dnp no) (property "Reference" "U1" (at 57.15 48.26 0) (effects (font (size 1.27 1.27)) (justify left bottom))) (property "Value" "AVR16DU28-I/SP" (at 82.55 48.26 0) (effects (font (size 1.27 1.27)) (justify right bottom))) (property "Footprint" "" (at 69.85 74.93 0) (effects (font (size 1.27 1.27)) (hide yes))) (property "Datasheet" "" (at 69.85 74.93 0) (effects (font (size 1.27 1.27)) (hide yes))) (property "Description" "AVR DU, SPDIP-28; pin numbers per DS40002576 I/O multiplexing table" (at 69.85 74.93 0) (effects (font (size 1.27 1.27)) (hide yes))) (pin "18")(pin "24")(pin "6")(pin "8")(pin "7")(pin "22")(pin "23")(pin "19")(pin "25")(pin "26")(pin "27")(pin "28")(pin "1")(pin "2")(pin "3")(pin "4")(pin "5")(pin "9")(pin "10")(pin "11")(pin "12")(pin "13")(pin "14")(pin "15")(pin "16")(pin "17")(pin "20")(pin "21") (instances (project "J48_RevI" (path "/ac26d7a1-d4c1-538e-978a-7250a60a85b4" (reference "U1") (unit 1)))))
+  (symbol (lib_id "GALProg:AVR16DU28") (at 69.85 74.93 0) (unit 1) (exclude_from_sim no) (in_bom yes) (on_board yes) (dnp no) (property "Reference" "U1" (at 57.15 48.26 0) (effects (font (size 1.27 1.27)) (justify left bottom))) (property "Value" "AVR16DU28-I/SP" (at 82.55 48.26 0) (effects (font (size 1.27 1.27)) (justify right bottom))) (property "Footprint" "" (at 69.85 74.93 0) (effects (font (size 1.27 1.27)) (hide yes))) (property "Datasheet" "" (at 69.85 74.93 0) (effects (font (size 1.27 1.27)) (hide yes))) (property "Description" "AVR DU, SPDIP-28; pin numbers per DS40002576 section 2.4 (SPDIP/SSOP-28 pinout)" (at 69.85 74.93 0) (effects (font (size 1.27 1.27)) (hide yes))) (pin "14")(pin "20")(pin "2")(pin "4")(pin "3")(pin "18")(pin "19")(pin "15")(pin "21")(pin "22")(pin "23")(pin "24")(pin "25")(pin "26")(pin "27")(pin "28")(pin "1")(pin "5")(pin "6")(pin "7")(pin "8")(pin "9")(pin "10")(pin "11")(pin "12")(pin "13")(pin "16")(pin "17") (instances (project "J48_RevI" (path "/ac26d7a1-d4c1-538e-978a-7250a60a85b4" (reference "U1") (unit 1)))))
   (symbol (lib_id "GALProg:R") (at 15.24 154.94 0) (unit 1) (exclude_from_sim no) (in_bom yes) (on_board yes) (dnp no) (property "Reference" "R1" (at 17.78 154.305 0) (effects (font (size 1.27 1.27)) (justify left))) (property "Value" "100" (at 17.78 156.21 0) (effects (font (size 1.27 1.27)) (justify left))) (property "Footprint" "" (at 15.24 154.94 0) (effects (font (size 1.27 1.27)) (hide yes))) (property "Datasheet" "" (at 15.24 154.94 0) (effects (font (size 1.27 1.27)) (hide yes))) (property "Description" "" (at 15.24 154.94 0) (effects (font (size 1.27 1.27)) (hide yes))) (pin "1")(pin "2") (instances (project "J48_RevI" (path "/ac26d7a1-d4c1-538e-978a-7250a60a85b4" (reference "R1") (unit 1)))))
   (symbol (lib_id "GALProg:R") (at 30.48 154.94 0) (unit 1) (exclude_from_sim no) (in_bom yes) (on_board yes) (dnp no) (property "Reference" "R2" (at 33.02 154.305 0) (effects (font (size 1.27 1.27)) (justify left))) (property "Value" "100" (at 33.02 156.21 0) (effects (font (size 1.27 1.27)) (justify left))) (property "Footprint" "" (at 30.48 154.94 0) (effects (font (size 1.27 1.27)) (hide yes))) (property "Datasheet" "" (at 30.48 154.94 0) (effects (font (size 1.27 1.27)) (hide yes))) (property "Description" "" (at 30.48 154.94 0) (effects (font (size 1.27 1.27)) (hide yes))) (pin "1")(pin "2") (instances (project "J48_RevI" (path "/ac26d7a1-d4c1-538e-978a-7250a60a85b4" (reference "R2") (unit 1)))))
